Commit message: control of wheels

File: src/twip_description/urdf/twip.urdf.xacro (robot description, xacro)
@@ -106,3 +106,35 @@
         <axis xyz="1 0 0" />
     </joint>
+    <!-- IMU -->
+    <link name="imu_link">
+        <inertial>
+            <origin xyz="-0.00552433659106688 0.000168210391520346 0.000514000497342681" rpy="0 0 0" />
+            <mass value="0.000528415362211671" />
+            <inertia ixx="1.46176048428261E-08" ixy="1.40015117949421E-10"
+                ixz="-1.99633872937403E-12"
+                iyy="8.59662482954888E-09" iyz="7.52375112767959E-12"
+                izz="2.30279421279312E-08" />
+        </inertial>
+        <visual>
+            <origin xyz="0 0 0" rpy="0 0 0" />
+            <geometry>
+                <mesh filename="package://twip_description/meshes/imu_link.STL" />
+            </geometry>
+            <material name="">
+                <color rgba="0.792156862745098 0.819607843137255 0.933333333333333 1" />
+            </material>
+        </visual>
+        <collision>
+            <origin xyz="0 0 0" rpy="0 0 0" />
+            <geometry>
+                <mesh filename="package://twip_description/meshes/imu_link.STL" />
+            </geometry>
+        </collision>
+    </link>
+    <joint name="imu_joint" type="fixed">
+        <origin xyz="-0.0005 0 0.125" rpy="1.5708 1.6057  0" />
+        <parent link="base_link" />
+        <child link="imu_link" />
+        <axis xyz="0 0 0" />
+    </joint>
 </robot>

File: src/twip_description/urdf/twip_gazebo.xacro (robot description, xacro)
@@ -27,4 +27,6 @@
         <parameters>$(find twip_controller)/config/twip_controllers.yaml</parameters>
       </plugin>
+      <plugin filename="ignition-gazebo-imu-system" name="ignition::gazebo::systems::Imu">
+      </plugin>
     </xacro:if>
     <!-- ROS 2 Iron or above -->
@@ -33,5 +35,59 @@
         <parameters>$(find twip_controller)/config/twip_controllers.yaml</parameters>
       </plugin>
+      <plugin filename="gz-sim-imu-system" name="gz::sim::systems::Imu">
+      </plugin>
     </xacro:unless>
   </gazebo>
+  <gazebo reference="imu_link">
+    <sensor name="imu" type="imu">
+      <alwaysOn>true</alwaysOn>
+      <updateRate>100.0</updateRate>
+      <gz_frame_id>imu_link</gz_frame_id>
+      <topic>imu</topic>
+      <imu>
+        <noise>
+          <angular_velocity>
+            <x>
+              <noise type="gaussian">
+                <mean>0.0</mean>
+                <stddev>2e-4</stddev>
+              </noise>
+            </x>
+            <y>
+              <noise type="gaussian">
+                <mean>0.0</mean>
+                <stddev>2e-4</stddev>
+              </noise>
+            </y>
+            <z>
+              <noise type="gaussian">
+                <mean>0.0</mean>
+                <stddev>2e-4</stddev>
+              </noise>
+            </z>
+          </angular_velocity>
+          <linear_acceleration>
+            <x>
+              <noise type="gaussian">
+                <mean>0.0</mean>
+                <stddev>0.017</stddev>
+              </noise>
+            </x>
+            <y>
+              <noise type="gaussian">
+                <mean>0.0</mean>
+                <stddev>0.017</stddev>
+              </noise>
+            </y>
+            <z>
+              <noise type="gaussian">
+                <mean>0.0</mean>
+                <stddev>0.017</stddev>
+              </noise>
+            </z>
+          </linear_acceleration>
+        </noise>
+      </imu>
+    </sensor>
+  </gazebo>
 </robot>

Commit message: fix kalman

File: src/twip_description/urdf/twip.urdf.xacro (robot description, xacro)
@@ -117,5 +117,5 @@
         </inertial>
         <visual>
-            <origin xyz="0 0 0" rpy="0 0 0" />
+            <origin xyz="-0.0005 0 0" rpy="1.5708 1.6057  0" />
             <geometry>
                 <mesh filename="package://twip_description/meshes/imu_link.STL" />
@@ -126,5 +126,5 @@
         </visual>
         <collision>
-            <origin xyz="0 0 0" rpy="0 0 0" />
+            <origin xyz="-0.0005 0 0" rpy="1.5708 1.6057  0" />
             <geometry>
                 <mesh filename="package://twip_description/meshes/imu_link.STL" />
@@ -133,5 +133,5 @@
     </link>
     <joint name="imu_joint" type="fixed">
-        <origin xyz="-0.0005 0 0.125" rpy="1.5708 1.6057  0" />
+        <origin xyz="0 0 0.125" rpy="0 0 0" />
         <parent link="base_link" />
         <child link="imu_link" />

Commit message: control with torques

File: src/twip_description/urdf/twip.urdf.xacro (robot description, xacro)
@@ -8,4 +8,13 @@
     <xacro:include filename="$(find twip_description)/urdf/twip_ros2_control.xacro" />
     <link name="base_footprint" />
+    <material name="blue">
+        <color rgba="0.125 0.384 0.702 1.0" />
+    </material>
+    <material name="grey">
+        <color rgba="0.5 0.5 0.5 1.0" />
+    </material>
+    <material name="dark_grey">
+        <color rgba="0.1 0.1 0.1 1.0" />
+    </material>
     <!-- Robot Body -->
     <link name="base_link">
@@ -26,4 +35,5 @@
                 <mesh filename="package://twip_description/meshes/robot_body.stl" />
             </geometry>
+            <material name="blue" />
         </visual>
         <collision>
@@ -57,15 +67,16 @@
                 <mesh filename="package://twip_description/meshes/right_wheel.stl" />
             </geometry>
+            <material name="dark_grey" />
         </visual>
         <collision>
             <origin xyz="0 0 0" rpy="0 0 0" />
             <geometry>
-                <!-- <mesh filename="package://twip_description/meshes/right_wheel.stl" /> -->
-                <sphere radius="0.0325" />
+                <mesh filename="package://twip_description/meshes/right_wheel.stl" />
+                <!-- <cylinder radius="0.0325" length="0.03" /> -->
             </geometry>
         </collision>
     </link>
     <joint name="wheel_right_joint" type="continuous">
-        <origin xyz="-0.078268 0 0.0325" rpy="0 0 0" />
+        <origin xyz="-0.07865 0 0.0325" rpy="0 0 0" />
         <parent
             link="base_link" />
@@ -91,15 +102,16 @@
                 <mesh filename="package://twip_description/meshes/left_wheel.stl" />
             </geometry>
+            <material name="dark_grey" />
         </visual>
         <collision>
             <origin xyz="0 0 0" rpy="0 0 0" />
             <geometry>
-                <!-- <mesh filename="package://twip_description/meshes/left_wheel.stl" /> -->
-                <sphere radius="0.0325" />
+                <mesh filename="package://twip_description/meshes/left_wheel.stl" />
+                <!-- <cylinder radius="0.0325" length="0.03" /> -->
             </geometry>
         </collision>
     </link>
     <joint name="wheel_left_joint" type="continuous">
-        <origin xyz="0.079032 0 0.0325" rpy="0 0 0" />
+        <origin xyz="0.07865 0 0.0325" rpy="0 0 0" />
         <parent link="base_link" />
         <child link="wheel_left_link" />
@@ -121,7 +133,5 @@
                 <mesh filename="package://twip_description/meshes/imu_link.STL" />
             </geometry>
-            <material name="">
-                <color rgba="0.792156862745098 0.819607843137255 0.933333333333333 1" />
-            </material>
+            <material name="grey" />
         </visual>
         <collision>

File: src/twip_description/urdf/twip_gazebo.xacro (robot description, xacro)
@@ -10,4 +10,8 @@
     <maxVel>0.1</maxVel> <!-- what units is this??? -->
     <fdir1>1 0 0</fdir1>
+    <provideFeedback>true</provideFeedback>
+    <implicitSpringDamper>true</implicitSpringDamper>
+    <selfCollide>true</selfCollide>
+    <dynamics damping="0.1" friction="0.05" />
   </gazebo>
   <gazebo reference="wheel_right_link">
@@ -17,6 +21,10 @@
     <kd>10.0</kd>
     <minDepth>0.001</minDepth>
-    <maxVel>0.1</maxVel>
+    <maxVel>0.1</maxVel> <!-- what units is this??? -->
     <fdir1>1 0 0</fdir1>
+    <provideFeedback>true</provideFeedback>
+    <implicitSpringDamper>true</implicitSpringDamper>
+    <selfCollide>true</selfCollide>
+    <dynamics damping="0.1" friction="0.05" />
   </gazebo>
   <!-- ROS 2 Control -->
@@ -26,4 +34,6 @@
       <plugin filename="ign_ros2_control-system" name="ign_ros2_control::IgnitionROS2ControlPlugin">
         <parameters>$(find twip_controller)/config/twip_controllers.yaml</parameters>
+        <robot_param>robot_description</robot_param>
+        <robot_param_node>robot_state_publisher</robot_param_node>
       </plugin>
       <plugin filename="ignition-gazebo-imu-system" name="ignition::gazebo::systems::Imu">
@@ -34,4 +44,6 @@
       <plugin filename="gz_ros2_control-system" name="gz_ros2_control::GazeboSimROS2ControlPlugin">
         <parameters>$(find twip_controller)/config/twip_controllers.yaml</parameters>
+        <robot_param>robot_description</robot_param>
+        <robot_param_node>robot_state_publisher</robot_param_node>
       </plugin>
       <plugin filename="gz-sim-imu-system" name="gz::sim::systems::Imu">
@@ -39,55 +51,7 @@
     </xacro:unless>
   </gazebo>
+  <!-- El resto de tu configuración IMU permanece igual -->
   <gazebo reference="imu_link">
-    <sensor name="imu" type="imu">
-      <alwaysOn>true</alwaysOn>
-      <updateRate>100.0</updateRate>
-      <gz_frame_id>imu_link</gz_frame_id>
-      <topic>imu</topic>
-      <imu>
-        <noise>
-          <angular_velocity>
-            <x>
-              <noise type="gaussian">
-                <mean>0.0</mean>
-                <stddev>2e-4</stddev>
-              </noise>
-            </x>
-            <y>
-              <noise type="gaussian">
-                <mean>0.0</mean>
-                <stddev>2e-4</stddev>
-              </noise>
-            </y>
-            <z>
-              <noise type="gaussian">
-                <mean>0.0</mean>
-                <stddev>2e-4</stddev>
-              </noise>
-            </z>
-          </angular_velocity>
-          <linear_acceleration>
-            <x>
-              <noise type="gaussian">
-                <mean>0.0</mean>
-                <stddev>0.017</stddev>
-              </noise>
-            </x>
-            <y>
-              <noise type="gaussian">
-                <mean>0.0</mean>
-                <stddev>0.017</stddev>
-              </noise>
-            </y>
-            <z>
-              <noise type="gaussian">
-                <mean>0.0</mean>
-                <stddev>0.017</stddev>
-              </noise>
-            </z>
-          </linear_acceleration>
-        </noise>
-      </imu>
-    </sensor>
+    <!-- ... tu configuración IMU existente ... -->
   </gazebo>
 </robot>

File: src/twip_description/urdf/twip_ros2_control.xacro (robot description, xacro)
@@ -18,17 +18,27 @@
         <joint name="wheel_right_joint">
             <command_interface name="velocity">
-              <param name="min">-1</param>
-              <param name="max">1</param>
+                <param name="min">-1</param>
+                <param name="max">1</param>
+            </command_interface>
+            <command_interface name="effort">
+                <param name="min">-1</param>
+                <param name="max">1</param>
             </command_interface>
             <state_interface name="position" />
             <state_interface name="velocity" />
+            <state_interface name="effort" />
         </joint>
         <joint name="wheel_left_joint">
             <command_interface name="velocity">
-              <param name="min">-1</param>
-              <param name="max">1</param>
+                <param name="min">-1</param>
+                <param name="max">1</param>
+            </command_interface>
+            <command_interface name="effort">
+                <param name="min">-1</param>
+                <param name="max">1</param>
             </command_interface>
             <state_interface name="position" />
             <state_interface name="velocity" />
+            <state_interface name="effort" />
         </joint>
     </ros2_control>
